Commit message: completed launch file

File: src/c_atm_description/urdf/atm.urdf (robot description, URDF)
Before this commit: robot atm, 5 links, 4 joints
Joints:
- joint baselink_lefttire: origin xyz=0.0 0.08 0.023 rpy=-1.57 0 0 -> xyz=0.0 -0.08 0.023 rpy=-1.57 0 0
- joint baselink_righttire: origin xyz=0.0 -0.080 0.023 rpy=-1.57 0 0 -> xyz=0.0 0.080 0.023 rpy=-1.57 0 0
